Commit message: tried to do prismatic joint, didnt work

File: src/robutler_description/urdf/robutler(prismatic).urdf.xacro (robot description, xacro)
@@ -195,7 +195,7 @@
   <link name="antenna_link">
     <visual>
-      <origin xyz="0 0 0.75" rpy="0 0 0"/>
-      <geometry>
-        <cylinder length="1.5" radius="0.003"/>
+      <origin xyz="0 0 0.1" rpy="0 0 0"/>
+      <geometry>
+        <cylinder length="0.2" radius="0.003"/>
       </geometry>
       <material name="dark"/>
@@ -212,9 +212,10 @@
   </link>
   <!-- joint between the top of the antenna and the camera joints -->
- <joint name="antenna_camera_joint" type="fixed">
+ <joint name="antenna_camera_joint" type="prismatic">
     <parent link="antenna_link"/>
     <child link="antena_camera_link"/>
-    <origin xyz="0 0 1.5" rpy="0 0 0"/>
+    <origin xyz="0 0 0.2" rpy="0 0 0"/>
     <axis xyz="0 0 1"/>
+    <limit lower="0" upper="1.3" effort="0" velocity="0"/>
   </joint>
   <joint name="camera_joint_a" type="fixed">
