Commit message: 3 xacro files. main, prismatic and 2 cameras

File: src/robutler_description/urdf/robutler_2_cameras.urdf.xacro (robot description, xacro)
@@ -3,4 +3,8 @@
   <xacro:include filename="$(find robutler_description)/urdf/common_properties.xacro"/>
   <xacro:include filename="$(find robutler_description)/urdf/robutler.gazebo.xacro"/>
+  <!--
+    This file is to display the extra camera in use in the robutler robot. However, not double cameras are used to do any functions, only one
+      making this urdf file not usable in our main project.
+    -->
   <link name="base_footprint"/>
   <joint name="base_joint" type="fixed">
@@ -161,4 +165,29 @@
     </inertial>
   </link>
+  <joint name="camera_joint" type="fixed">
+    <origin xyz="0.073 -0.011 0.084" rpy="0 0 0"/>
+    <parent link="base_link"/>
+    <child link="camera_link"/>
+  </joint>
+  <link name="camera_link">
+    <collision>
+      <origin xyz="0.005 0.011 0.013" rpy="0 0 0"/>
+      <geometry>
+        <box size="0.015 0.030 0.027"/>
+      </geometry>
+    </collision>
+  </link>
+  <joint name="camera_rgb_joint" type="fixed">
+    <origin xyz="0.003 0.011 0.009" rpy="0 0 0"/>
+    <parent link="camera_link"/>
+    <child link="camera_rgb_frame"/>
+  </joint>
+  <link name="camera_rgb_frame"/>
+  <joint name="camera_rgb_optical_joint" type="fixed">
+    <origin xyz="0 0 0" rpy="-1.57 0 -1.57"/>
+    <parent link="camera_rgb_frame"/>
+    <child link="camera_rgb_optical_frame"/>
+  </joint>
+  <link name="camera_rgb_optical_frame"/>
   <joint name="antenna_for_camera" type="fixed">
     <parent link="base_link"/>
@@ -182,5 +211,5 @@
         <origin xyz="0 0 0 " rpy="0 0 0"/>
         <geometry>
-          <sphere radius="0.01"/>
+          <sphere radius="0.001"/>
         </geometry>
       </visual>
@@ -193,30 +222,49 @@
     <axis xyz="0 0 1"/>
   </joint>
-  <joint name="camera_joint_antena" type="fixed">
+  <joint name="camera_joint_a" type="fixed">
     <parent link="antena_camera_link"/>
-    <child link="camera_link"/>
+    <child link="camera_link_a"/>
     <axis xyz="0 0 1 " />
     <origin xyz="0 0 0 " rpy="0 0 0"/>
   </joint>
   <!-- camera links, joints and camera params  -->
-  <link name="camera_link">
-    <collision>
-      <origin xyz="0.005 0.011 0.013" rpy="0 0 0"/>
-      <geometry>
-        <box size="0.015 0.030 0.027"/>
-      </geometry>
-    </collision>
-  </link>
-  <joint name="camera_rgb_joint" type="fixed">
-    <origin xyz="0.003 0.011 0.009" rpy="0 0 0"/>
-    <parent link="camera_link"/>
-    <child link="camera_rgb_frame"/>
-  </joint>
-  <link name="camera_rgb_frame"/>
-  <joint name="camera_rgb_optical_joint" type="fixed">
-    <origin xyz="0 0 0" rpy="-1.57 0 -1.57"/>
-    <parent link="camera_rgb_frame"/>
-    <child link="camera_rgb_optical_frame"/>
-  </joint>
-  <link name="camera_rgb_optical_frame"/>
+  <link name="camera_link_a">
+    <visual>
+        <geometry>
+            <sphere radius="0.01"/>
+        </geometry>
+        <material name="red"/>
+    </visual>
+  </link>
+  <joint name="camera_optical_joint" type="fixed">
+      <parent link="camera_link_a"/>
+      <child link="camera_link_optical"/>
+      <axis xyz="0 0 1"/>
+      <origin xyz="0 0 0" rpy= "-1.57 0 -1.57"/>
+  </joint>
+  <!-- "${-pi/2} 0 ${-pi/2}" -->
+  <link name="camera_link_optical"></link>
+  <gazebo reference="camera_link_a">
+      <material>Gazebo/Red</material>
+        <sensor name="camera" type="camera">
+            <pose> 0 0 0 0 0 0 </pose>
+            <!-- <visualize>true</visualize> -->
+            <update_rate>60</update_rate>
+            <camera>
+                <horizontal_fov>1.089</horizontal_fov>
+                <image>
+                    <format>R8G8B8</format>
+                    <width>640</width>
+                    <height>480</height>
+                </image>
+                <clip>
+                    <near>0.05</near>
+                    <far>8.0</far>
+                </clip>
+            </camera>
+            <plugin name="camera_controller" filename="libgazebo_ros_camera.so">
+                <frame_name>camera_link_optical</frame_name>
+            </plugin>
+        </sensor>
+  </gazebo>
 </robot>

File: src/robutler_description/urdf/robutler_prismatic_joint.urdf.xacro (robot description, xacro)
@@ -3,4 +3,8 @@
   <xacro:include filename="$(find robutler_description)/urdf/common_properties.xacro"/>
   <xacro:include filename="$(find robutler_description)/urdf/robutler.gazebo.xacro"/>
+  <!--  REQUIRES  joint_state_publisher_gui to run the prismatic joint manually. no automatic functions to move the camera yet.
+    This file is to be used to display the use of a prismatic joint, that doesnt allow to see the values of the new camera due to the all of the
+      parents of said camera need to be fixed
+   -->
   <link name="base_footprint"/>
   <joint name="base_joint" type="fixed">
@@ -161,4 +165,29 @@
     </inertial>
   </link>
+  <joint name="camera_joint" type="fixed">
+    <origin xyz="0.073 -0.011 0.084" rpy="0 0 0"/>
+    <parent link="base_link"/>
+    <child link="camera_link"/>
+  </joint>
+  <link name="camera_link">
+    <collision>
+      <origin xyz="0.005 0.011 0.013" rpy="0 0 0"/>
+      <geometry>
+        <box size="0.015 0.030 0.027"/>
+      </geometry>
+    </collision>
+  </link>
+  <joint name="camera_rgb_joint" type="fixed">
+    <origin xyz="0.003 0.011 0.009" rpy="0 0 0"/>
+    <parent link="camera_link"/>
+    <child link="camera_rgb_frame"/>
+  </joint>
+  <link name="camera_rgb_frame"/>
+  <joint name="camera_rgb_optical_joint" type="fixed">
+    <origin xyz="0 0 0" rpy="-1.57 0 -1.57"/>
+    <parent link="camera_rgb_frame"/>
+    <child link="camera_rgb_optical_frame"/>
+  </joint>
+  <link name="camera_rgb_optical_frame"/>
   <joint name="antenna_for_camera" type="fixed">
     <parent link="base_link"/>
@@ -170,7 +199,7 @@
   <link name="antenna_link">
     <visual>
-      <origin xyz="0 0 0.75" rpy="0 0 0"/>
-      <geometry>
-        <cylinder length="1.5" radius="0.003"/>
+      <origin xyz="0 0 0.1" rpy="0 0 0"/>
+      <geometry>
+        <cylinder length="0.2" radius="0.003"/>
       </geometry>
       <material name="dark"/>
@@ -182,41 +211,59 @@
         <origin xyz="0 0 0 " rpy="0 0 0"/>
         <geometry>
-          <sphere radius="0.01"/>
+          <sphere radius="0.001"/>
         </geometry>
       </visual>
   </link>
   <!-- joint between the top of the antenna and the camera joints -->
- <joint name="antenna_camera_joint" type="fixed">
+ <joint name="antenna_camera_joint" type="prismatic">
     <parent link="antenna_link"/>
     <child link="antena_camera_link"/>
-    <origin xyz="0 0 1.5" rpy="0 0 0"/>
+    <origin xyz="0 0 0.2" rpy="0 0 0"/>
     <axis xyz="0 0 1"/>
-  </joint>
-  <joint name="camera_joint_antena" type="fixed">
+    <limit lower="0" upper="1.3" effort="0" velocity="0"/>
+  </joint>
+  <joint name="camera_joint_a" type="fixed">
     <parent link="antena_camera_link"/>
-    <child link="camera_link"/>
+    <child link="camera_link_a"/>
     <axis xyz="0 0 1 " />
     <origin xyz="0 0 0 " rpy="0 0 0"/>
   </joint>
   <!-- camera links, joints and camera params  -->
-  <link name="camera_link">
-    <collision>
-      <origin xyz="0.005 0.011 0.013" rpy="0 0 0"/>
-      <geometry>
-        <box size="0.015 0.030 0.027"/>
-      </geometry>
-    </collision>
-  </link>
-  <joint name="camera_rgb_joint" type="fixed">
-    <origin xyz="0.003 0.011 0.009" rpy="0 0 0"/>
-    <parent link="camera_link"/>
-    <child link="camera_rgb_frame"/>
-  </joint>
-  <link name="camera_rgb_frame"/>
-  <joint name="camera_rgb_optical_joint" type="fixed">
-    <origin xyz="0 0 0" rpy="-1.57 0 -1.57"/>
-    <parent link="camera_rgb_frame"/>
-    <child link="camera_rgb_optical_frame"/>
-  </joint>
-  <link name="camera_rgb_optical_frame"/>
+    <link name="camera_link_a">
+        <visual>
+            <geometry>
+                <box size="0.010 0.03 0.03"/>
+            </geometry>
+            <material name="red"/>
+        </visual>
+    </link>
+    <joint name="camera_optical_joint" type="fixed">
+        <parent link="camera_link_a"/>
+        <child link="camera_link_optical"/>
+        <origin xyz="0 0 0" rpy="${-pi/2} 0 ${-pi/2}"/>
+    </joint>
+    <link name="camera_link_optical"></link>
+    <gazebo reference="camera_link_a">
+        <material>Gazebo/Red</material>
+        <sensor name="camera" type="camera">
+            <pose> 0 0 0 0 0 0 </pose>
+            <visualize>true</visualize>
+            <update_rate>10</update_rate>
+            <camera>
+                <horizontal_fov>1.089</horizontal_fov>
+                <image>
+                    <format>R8G8B8</format>
+                    <width>640</width>
+                    <height>480</height>
+                </image>
+                <clip>
+                    <near>0.05</near>
+                    <far>8.0</far>
+                </clip>
+            </camera>
+            <plugin name="camera_controller" filename="libgazebo_ros_camera.so">
+                <frame_name>camera_link_optical</frame_name>
+            </plugin>
+        </sensor>
+    </gazebo>
 </robot>
