Commit message: change robutler xacro to elevate camera

File: src/robutler_description/urdf/robutler.urdf.xacro (robot description, xacro)
@@ -163,5 +163,5 @@
   <joint name="camera_joint" type="fixed">
     <!-- <origin xyz="0.073 -0.011 0.084" rpy="0 0 0"/> -->
-    <origin xyz="0.073 -0.011 1" rpy="0 0 0"/>
+    <origin xyz="0.073 -0.011 1.5" rpy="0 0 0"/>
     <parent link="base_link"/>
     <child link="camera_link"/>

Commit message: nova camera- com 50cm altura

File: src/robutler_description/urdf/robutler.urdf.xacro (robot description, xacro)
@@ -162,6 +162,5 @@
   </link>
   <joint name="camera_joint" type="fixed">
-    <!-- <origin xyz="0.073 -0.011 0.084" rpy="0 0 0"/> -->
-    <origin xyz="0.073 -0.011 1.5" rpy="0 0 0"/>
+    <origin xyz="0.073 -0.011 0.084" rpy="0 0 0"/>
     <parent link="base_link"/>
     <child link="camera_link"/>
@@ -187,3 +186,101 @@
   </joint>
   <link name="camera_rgb_optical_frame"/>
+  <joint name="antenna_for_camera" type="fixed">
+    <parent link="base_link"/>
+    <child link="antenna_link"/>
+    <axis xyz="0 1 0"/>
+    <origin xyz="-0.1325 0 0.09" rpy="0 0 0"/>
+  </joint>
+  <link name="antenna_link">
+    <visual>
+      <origin xyz="0 0 0.25" rpy="0 0 0"/>
+      <geometry>
+        <cylinder length="0.5" radius="0.003"/>
+      </geometry>
+      <material name="dark"/>
+    </visual>
+<!--
+    <collision>
+      <origin xyz="0 0 0" rpy="0 0 0"/>
+        <geometry>
+          <cylinder length="0.5" radius="0.003"/>
+        </geometry>
+    </collision>
+    <inertial>
+      <mass value="1.0e-100" />
+      <origin xyz="0 0 0" />
+      <inertia ixx="0.001" ixy="0.0" ixz="0.0"
+               iyy="0.001" iyz="0.0"
+               izz="0.001" />
+    </inertial> -->
+  </link>
+  <link name="antena_camera_link">
+      <visual>
+        <origin xyz="0 0 0 " rpy="0 0 0"/>
+        <geometry>
+          <sphere radius="0.001"/>
+        </geometry>
+      </visual>
+  </link>
+    <!-- Add joint to connect camera to base_link -->
+  <joint name="antenna_camera_joint" type="fixed">
+    <parent link="antenna_link"/>
+    <child link="antena_camera_link"/>
+    <origin xyz="0 0 0.5" rpy="0 0 0"/>
+  </joint>
+  <joint name="camera_joint_a" type="fixed">
+    <parent link="antena_camera_link"/>
+    <child link="camera_link_a"/>
+    <origin xyz="0 0 0" rpy="0 0 0"/>
+  </joint>
+  <link name="camera_link_a">
+    <visual>
+        <geometry>
+            <sphere radius="0.01"/>
+        </geometry>
+        <material name="red"/>
+    </visual>
+    <!-- <collision>
+        <geometry>
+            <sphere radius="0.01"/>
+        </geometry>
+    </collision>
+    <inertial>
+      <mass value="1e-100" />
+      <origin xyz="0 0 0" />
+      <inertia ixx="0.001" ixy="0.0" ixz="0.0"
+               iyy="0.001" iyz="0.0"
+               izz="0.001" />
+    </inertial> -->
+  </link>
+      <joint name="camera_optical_joint" type="fixed">
+          <parent link="camera_link_a"/>
+          <child link="camera_link_optical"/>
+          <origin xyz="0 0 0" rpy= "-1.57 0 -1.57"/>
+      </joint>
+  <!-- "${-pi/2} 0 ${-pi/2}" -->
+      <link name="camera_link_optical"></link>
+  <gazebo reference="camera_link_a">
+      <material>Gazebo/Red</material>
+        <sensor name="camera" type="camera">
+            <pose> 0 0 0 0 0 0 </pose>
+            <!-- <visualize>true</visualize> -->
+            <update_rate>60</update_rate>
+            <camera>
+                <horizontal_fov>1.089</horizontal_fov>
+                <image>
+                    <format>R8G8B8</format>
+                    <width>640</width>
+                    <height>480</height>
+                </image>
+                <clip>
+                    <near>0.05</near>
+                    <far>8.0</far>
+                </clip>
+            </camera>
+            <plugin name="camera_controller" filename="libgazebo_ros_camera.so">
+                <frame_name>camera_link_optical</frame_name>
+            </plugin>
+        </sensor>
+  </gazebo>
 </robot>

Commit message: braço com 1.5m de altura, sem colisoes e peso

File: src/robutler_description/urdf/robutler.urdf.xacro (robot description, xacro)
@@ -194,7 +194,7 @@
   <link name="antenna_link">
     <visual>
-      <origin xyz="0 0 0.25" rpy="0 0 0"/>
-      <geometry>
-        <cylinder length="0.5" radius="0.003"/>
+      <origin xyz="0 0 0.75" rpy="0 0 0"/>
+      <geometry>
+        <cylinder length="1.5" radius="0.003"/>
       </geometry>
       <material name="dark"/>
@@ -227,5 +227,5 @@
     <parent link="antenna_link"/>
     <child link="antena_camera_link"/>
-    <origin xyz="0 0 0.5" rpy="0 0 0"/>
+    <origin xyz="0 0 1.5" rpy="0 0 0"/>
   </joint>
   <joint name="camera_joint_a" type="fixed">

Commit message: Revert "New camera setup"

File: src/robutler_description/urdf/robutler.urdf.xacro (robot description, xacro)
@@ -162,5 +162,6 @@
   </link>
   <joint name="camera_joint" type="fixed">
-    <origin xyz="0.073 -0.011 0.084" rpy="0 0 0"/>
+    <!-- <origin xyz="0.073 -0.011 0.084" rpy="0 0 0"/> -->
+    <origin xyz="0.073 -0.011 1.5" rpy="0 0 0"/>
     <parent link="base_link"/>
     <child link="camera_link"/>
@@ -186,81 +187,3 @@
   </joint>
   <link name="camera_rgb_optical_frame"/>
-  <joint name="antenna_for_camera" type="fixed">
-    <parent link="base_link"/>
-    <child link="antenna_link"/>
-    <axis xyz="0 1 0"/>
-    <origin xyz="-0.1325 0 0.09" rpy="0 0 0"/>
-  </joint>
-  <!-- base / tube of the antenna -->
-  <link name="antenna_link">
-    <visual>
-      <origin xyz="0 0 0.75" rpy="0 0 0"/>
-      <geometry>
-        <cylinder length="1.5" radius="0.003"/>
-      </geometry>
-      <material name="dark"/>
-    </visual>
-  </link>
-  <!-- top of the antenna -->
-  <link name="antena_camera_link">
-      <visual>
-        <origin xyz="0 0 0 " rpy="0 0 0"/>
-        <geometry>
-          <sphere radius="0.001"/>
-        </geometry>
-      </visual>
-  </link>
-  <!-- joint between the top of the antenna and the camera joints -->
- <joint name="antenna_camera_joint" type="fixed">
-    <parent link="antenna_link"/>
-    <child link="antena_camera_link"/>
-    <origin xyz="0 0 1.5" rpy="0 0 0"/>
-    <axis xyz="0 0 1"/>
-  </joint>
-  <joint name="camera_joint_a" type="fixed">
-    <parent link="antena_camera_link"/>
-    <child link="camera_link_a"/>
-    <axis xyz="0 0 1 " />
-    <origin xyz="0 0 0 " rpy="0 0 0"/>
-  </joint>
-  <!-- camera links, joints and camera params  -->
-  <link name="camera_link_a">
-    <visual>
-        <geometry>
-            <sphere radius="0.01"/>
-        </geometry>
-        <material name="red"/>
-    </visual>
-  </link>
-  <joint name="camera_optical_joint" type="fixed">
-      <parent link="camera_link_a"/>
-      <child link="camera_link_optical"/>
-      <axis xyz="0 0 1"/>
-      <origin xyz="0 0 0" rpy= "-1.57 0 -1.57"/>
-  </joint>
-  <!-- "${-pi/2} 0 ${-pi/2}" -->
-  <link name="camera_link_optical"></link>
-  <gazebo reference="camera_link_a">
-      <material>Gazebo/Red</material>
-        <sensor name="camera" type="camera">
-            <pose> 0 0 0 0 0 0 </pose>
-            <!-- <visualize>true</visualize> -->
-            <update_rate>60</update_rate>
-            <camera>
-                <horizontal_fov>1.089</horizontal_fov>
-                <image>
-                    <format>R8G8B8</format>
-                    <width>640</width>
-                    <height>480</height>
-                </image>
-                <clip>
-                    <near>0.05</near>
-                    <far>8.0</far>
-                </clip>
-            </camera>
-            <plugin name="camera_controller" filename="libgazebo_ros_camera.so">
-                <frame_name>camera_link_optical</frame_name>
-            </plugin>
-        </sensor>
-  </gazebo>
 </robot>

Commit message: camera com angulo 10º

File: src/robutler_description/urdf/robutler.urdf.xacro (robot description, xacro)
@@ -209,9 +209,9 @@
   </link>
   <joint name="camera_rgb_joint" type="fixed">
-    <origin xyz="0.003 0.011 0.009" rpy="0 0 0"/>
+    <origin xyz="0.003 0.011 0.009" rpy="0  0.174532925 0"/>
     <parent link="camera_link"/>
     <child link="camera_rgb_frame"/>
   </joint>
-  <link name="camera_rgb_frame"/>
+  <link name="camera_rgb_frame" />
   <joint name="camera_rgb_optical_joint" type="fixed">
     <origin xyz="0 0 0" rpy="-1.57 0 -1.57"/>
